File: kicad/synth.kicad_sch (KiCad schematic)
At the start: 2 parts, among them U1 STM32F401RCTx

Commit message: Stereo schematic, code cleanup
Connections:
- net Analog Right Out: no longer names the net of U1.35 (PB14)
- net DAC Right Off: no longer names the net of U1.36 (PB15)
Other:
- removed sheet DAC
Changed lines of the file:
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@@
 	(wire
 		(pts
-			(xy 59.69 111.76) (xy 57.15 111.76)
+			(xy 62.23 25.4) (xy 57.15 25.4)
 		)
 		(stroke
@@
 	(wire
 		(pts
-			(xy 62.23 25.4) (xy 57.15 25.4)
+			(xy 58.42 35.56) (xy 57.15 35.56)
 		)
 		(stroke
@@
 	(wire
 		(pts
-			(xy 59.69 114.3) (xy 57.15 114.3)
+			(xy 41.91 121.92) (xy 41.91 123.19)
 		)
 		(stroke
@@
 	(wire
 		(pts
-			(xy 58.42 35.56) (xy 57.15 35.56)
+			(xy 36.83 25.4) (xy 49.53 25.4)
 		)
 		(stroke
@@
 	(wire
 		(pts
-			(xy 41.91 121.92) (xy 41.91 123.19)
+			(xy 39.37 121.92) (xy 39.37 123.19)
 		)
 		(stroke
@@
 		)
 	)
-	(wire
-		(pts
-			(xy 36.83 25.4) (xy 49.53 25.4)
-		)
-		(stroke
-			(width 0)
-			(type default)
-		)
-	)
-	(wire
-		(pts
-			(xy 39.37 121.92) (xy 39.37 123.19)
-		)
-		(stroke
-			(width 0)
-			(type default)
-		)
-	)
-	(label "Analog Right Out"
-		(at 59.69 111.76 0)
-		(effects
-			(font
-				(size 1.27 1.27)
-			)
-			(justify left bottom)
-		)
-	)
 	(label "DAC Right PWM"
 		(at 59.69 109.22 0)
-		(effects
-			(font
-				(size 1.27 1.27)
-			)
-			(justify left bottom)
-		)
-	)
-	(label "DAC Right Off"
-		(at 59.69 114.3 0)
 		(effects
 			(font
@@
 	)
 	(sheet
-		(at 86.36 38.1)
+		(at 99.06 25.4)
 		(size 52.07 12.7)
 		(exclude_from_sim no)
@@
 		)
 		(property "Sheetname" "DAC P-Channel"
-			(at 86.36 37.3884 0)
+			(at 99.06 24.6884 0)
 			(show_name no)
 			(do_not_autoplace no)
@@
 		)
 		(property "Sheetfile" "dac-pchannel.kicad_sch"
-			(at 86.36 51.3846 0)
+			(at 99.06 38.6846 0)
 			(show_name no)
 			(do_not_autoplace no)
@@
 		)
 		(property "Field2" ""
-			(at 86.36 38.1 0)
+			(at 99.06 25.4 0)
 			(hide yes)
 			(show_name no)
@@
 				)
 			)
-		)
-	)
-	(sheet
-		(at 86.36 20.32)
-		(size 52.07 12.7)
-		(exclude_from_sim no)
-		(in_bom yes)
-		(on_board yes)
-		(dnp no)
-		(fields_autoplaced yes)
-		(stroke
-			(width 0.1524)
-			(type solid)
-		)
-		(fill
-			(color 0 0 0 0)
-		)
-		(property "Sheetname" "DAC"
-			(at 86.36 19.6084 0)
-			(show_name no)
-			(do_not_autoplace no)
-			(effects
-				(font
-					(size 1.27 1.27)
-				)
-				(justify left bottom)
-			)
-		)
-		(property "Sheetfile" "CMOS-ADC.kicad_sch"
-			(at 86.36 33.6046 0)
-			(show_name no)
-			(do_not_autoplace no)
-			(effects
-				(font
-					(size 1.27 1.27)
-				)
-				(justify left top)
-			)
-		)
-		(instances
-			(project "synth"
-				(path "/1e7814a7-1315-4eb0-a9cb-3b93c6dc7966"
-					(page "4")
-				)
-			)
